File: ControllerPCB/ControllerPCB.kicad_sch (KiCad schematic)
At the start: 47 parts, among them J1 2x4 Pickup Conn, J10 Conn_01x03_Pin, J11 Conn_01x03_Pin, J12 Conn_01x03_Pin, J2 Conn_01x03_Pin, J3 USB_B_Micro, J4 10-pin SWD Connector, J5 1x4 String Output Conn, J6 2x20 Conn_1, J7 2x20 Conn_2, J8 Conn_01x03_Pin, J9 Conn_01x03_Pin, SW1 SW_SPDT, U2 STM32F439ZIT6, Y1 8MHz

Commit message: Began the PCB. Placed the decoupling caps, usb micro b conn and others. Adding footprints for components as well.
Parts:
- removed C19: 10n, Capacitor_SMD:C_01005_0402Metric, symbol Device:C
- removed C20: 1u, Capacitor_SMD:C_01005_0402Metric, symbol Device:C
- removed D2: D-_TVS, symbol Device:D_TVS
- removed D3: D+_TVS, symbol Device:D_TVS
- removed D4: VBUS_TVS, symbol Device:D_TVS
- removed J4: 10-pin SWD Connector, symbol Connector_Generic:Conn_02x05_Odd_Even
- added D1: D+_TVS, PESD3V6Z1BCSFYL:PMEG3005AESFYL, symbol PESD3V6Z1BCSFYL:PESD3V6Z1BCSFYL
- added D2: VBUS_TVS, PESD5V5C1BLYL:PESD5V5C1BLYL, symbol PESD5V5C1BLYL:PESD5V5C1BLYL
- added D3: D-_TVS, PESD3V6Z1BCSFYL:PMEG3005AESFYL, symbol PESD3V6Z1BCSFYL:PESD3V6Z1BCSFYL
- added J4: 10-pin Debug Conn, FTSH_105_01_F_D_K:SAMTEC_FTSH-105-01-F-D-K, symbol FTSH-105-01-F-D-K:FTSH-105-01-F-D-K
- C10: renamed from C6; footprint Capacitor_SMD:C_01005_0402Metric -> Capacitor_SMD:C_0402_1005Metric
- C11: renamed from C7; footprint Capacitor_SMD:C_01005_0402Metric -> Capacitor_SMD:C_0402_1005Metric
- C12: renamed from C21; footprint Capacitor_SMD:C_01005_0402Metric -> Capacitor_SMD:C_0402_1005Metric
- C13: renamed from C8; footprint Capacitor_SMD:C_01005_0402Metric -> Capacitor_SMD:C_0402_1005Metric
- C14: renamed from C26; footprint Capacitor_SMD:C_01005_0402Metric -> Capacitor_SMD:C_0402_1005Metric
- C15: renamed from C3; footprint Capacitor_SMD:C_01005_0402Metric -> Capacitor_SMD:C_0402_1005Metric
- C16: renamed from C4; footprint Capacitor_SMD:C_01005_0402Metric -> Capacitor_SMD:C_0402_1005Metric
- C17: renamed from C27; footprint Capacitor_SMD:C_01005_0402Metric -> Capacitor_SMD:C_0402_1005Metric
- C18: renamed from C2; footprint Capacitor_SMD:C_01005_0402Metric -> Capacitor_SMD:C_0402_1005Metric
- C19: renamed from C1; footprint Capacitor_SMD:C_01005_0402Metric -> Capacitor_SMD:C_0402_1005Metric
- C2: renamed from C13; footprint Capacitor_SMD:C_01005_0402Metric -> Capacitor_SMD:C_0402_1005Metric
- C22: renamed from C15; footprint Capacitor_SMD:C_0603_1608Metric -> Capacitor_SMD:C_0402_1005Metric
- C23: renamed from C16; footprint Capacitor_SMD:C_01005_0402Metric -> Capacitor_SMD:C_0402_1005Metric
- C24: renamed from C17; footprint Capacitor_SMD:C_01005_0402Metric -> Capacitor_SMD:C_0402_1005Metric
- C3: renamed from C9; footprint Capacitor_SMD:C_01005_0402Metric -> Capacitor_SMD:C_0402_1005Metric
- C4: renamed from C10; footprint Capacitor_SMD:C_01005_0402Metric -> Capacitor_SMD:C_0402_1005Metric
- C5: renamed from C11; footprint Capacitor_SMD:C_01005_0402Metric -> Capacitor_SMD:C_0402_1005Metric
- C6: renamed from C18; footprint Capacitor_SMD:C_01005_0402Metric -> Capacitor_SMD:C_0402_1005Metric
- C7: renamed from C12; footprint Capacitor_SMD:C_01005_0402Metric -> Capacitor_SMD:C_0402_1005Metric
- C8: renamed from C22; footprint Capacitor_SMD:C_01005_0402Metric -> Capacitor_SMD:C_0402_1005Metric
- C9: renamed from C5; footprint Capacitor_SMD:C_01005_0402Metric -> Capacitor_SMD:C_0402_1005Metric
- FB1: footprint (none) -> Inductor_SMD:L_0603_1608Metric
- J1: renamed from J6; footprint (none) -> 75869-107LF:SHDR40W62P254_2X20_5801X920X957P
- J10: renamed from J12; footprint (none) -> 22292031:CONN_AE-6410-03A_MOL
- J11: renamed from J5; footprint (none) -> 22292041:CONN_AE-6410-04A_MOL
- J12: renamed from J1; footprint (none) -> 75869_332LF:AMPHENOL_75869-332LF
- J2, J9: footprint (none) -> 22292031:CONN_AE-6410-03A_MOL
- J3: renamed from J10; footprint (none) -> 22292031:CONN_AE-6410-03A_MOL
- J5: renamed from J8; footprint (none) -> 22292031:CONN_AE-6410-03A_MOL
- J6: renamed from J11; footprint (none) -> 22292031:CONN_AE-6410-03A_MOL
- J7: renamed from J3; footprint (none) -> Connector_USB:USB_Micro-B_Wuerth_629105150521
- J8: renamed from J7; footprint (none) -> 75869-107LF:SHDR40W62P254_2X20_5801X920X957P
- R3: renamed from R7; footprint (none) -> Resistor_SMD:R_0402_1005Metric
- R4: renamed from R8; footprint (none) -> Resistor_SMD:R_0402_1005Metric
- SW1: footprint (none) -> JS102011SAQN:SW_JS102011SAQN
- Y1: footprint (none) -> 830059082:830059082
- renumbered C14 to C1, R82 to R1, R1 to R2, U2 to U1
Connections:
- net +3.3V: now also J4.01
- net ADC_String_1: no longer U1.34 (PA0)
- net ADC_String_2: no longer U1.35 (PA1)
- net ADC_String_3: no longer U1.36 (PA2)
- net ADC_String_4: no longer U1.37 (PA3)
- net D+: now also D1.1
- net D-: now also D3.1
- net GND: now also D1.2, D2.2 (K2), D3.2, J4.03, J4.05, J4.09
- net NRST: now also J4.10
- net SWDCLK: now also J4.04
- net SWDIO: now also J4.02
- net SWO: now also J4.06
- net VCAP_1: now reaches C14.1, U1.71 (VCAP_1)
- net VBUS_TVS: now reaches J7.1 (VBUS), R3.1
- net VBUS_TVS: now also D2.1 (K1)
- net VCAP_2: now reaches C17.1, U1.106 (VCAP_2)
- net PG10 renamed String_1_out
- net PG11 renamed String_2_out
- net PG12 renamed String_3_out
- net PG13 renamed String_4_out
- new net ADC_String_1_F: U1.34 (PA0)
- new net ADC_String_2_F: U1.35 (PA1)
- new net ADC_String_3_F: U1.36 (PA2)
- new net ADC_String_4_F: U1.37 (PA3)
- no-connect marks 15 -> 16
Other:
- note added: "732-5960-1-ND"
- note added: "WM2745-ND"
- note removed: "23-0022111031-ND"
- note removed: "ESD351DPYR"
- note removed: "PESD5V5C1BLYL"
