File: ControllerPCB/ControllerPCB.kicad_sch (KiCad schematic)
At the start: 45 parts, among them J1 2x20 Conn_1, J10 Conn_01x03_Pin, J11 1x4 String Output Conn, J12 2x4 Pickup Conn, J2 Conn_01x03_Pin, J3 Conn_01x03_Pin, J4 10-pin Debug Conn, J5 Conn_01x03_Pin, J6 Conn_01x03_Pin, J7 USB_B_Micro, J8 2x20 Conn_2, J9 Conn_01x03_Pin, SW1 SW_SPDT, U1 STM32F439ZIT6, Y1 8MHz

Commit message: Added separate sheet for IO. Added TVS diodes for every external input to the controller except for the ADC and MIDI control inputs. Still need to add decoupling caps for the 9V humbucker source. Parts were chosen with JLPCB library stock in mind. Replaced the 8MHz crystal with a 16MHz crystal.
Parts:
- removed D1: D+_TVS, PESD3V6Z1BCSFYL:PMEG3005AESFYL, symbol PESD3V6Z1BCSFYL:PESD3V6Z1BCSFYL
- removed D2: VBUS_TVS, PESD5V5C1BLYL:PESD5V5C1BLYL, symbol PESD5V5C1BLYL:PESD5V5C1BLYL
- removed D3: D-_TVS, PESD3V6Z1BCSFYL:PMEG3005AESFYL, symbol PESD3V6Z1BCSFYL:PESD3V6Z1BCSFYL
- removed J1: 2x20 Conn_1, 75869-107LF:SHDR40W62P254_2X20_5801X920X957P, symbol Connector_Generic:Conn_02x20_Odd_Even
- removed J10: Conn_01x03_Pin, 22292031:CONN_AE-6410-03A_MOL, symbol Connector:Conn_01x03_Pin
- removed J11: 1x4 String Output Conn, 22292041:CONN_AE-6410-04A_MOL, symbol Connector:Conn_01x04_Pin
- removed J8: 2x20 Conn_2, 75869-107LF:SHDR40W62P254_2X20_5801X920X957P, symbol Connector_Generic:Conn_02x20_Odd_Even
- added C123: 100n, Capacitor_SMD:C_0402_1005Metric, symbol Device:C
- added D101, D102, D103, D104, D109, D110, D111, D112, D113, D114, D115, D116: D_TVS_Small, symbol Device:D_TVS_Small
- added D105, D106, D107, D108: D_Small, symbol Device:D_Small
- added J102: 1x4 String Output Conn, 22292041:CONN_AE-6410-04A_MOL, symbol Connector:Conn_01x04_Pin
- added R103, R104, R105, R106: 22R, symbol Device:R_Small
- Y101: renamed from Y1; value 8MHz -> 16MHz
- renumbered C1 to C101, C2 to C102, C3 to C103, C4 to C104, C5 to C105, C6 to C106, C7 to C107, C8 to C108, C9 to C109, C10 to C110, C11 to C111, C12 to C112, C13 to C113, C14 to C114, C15 to C115, C16 to C116, C17 to C117, C18 to C118, C19 to C119, C22 to C120, C23 to C121, C24 to C122, FB1 to FB101, J12 to J101, J2 to J103, J3 to J104, J5 to J105, J6 to J106, J7 to J107, J4 to J108, J9 to J109, R2 to R101, R1 to R102, R3 to R107, R4 to R108, SW1 to SW101, U1 to U101
Connections:
- net +3.3V: now also D116.2 (A2)
- net ADC_Mod: no longer J105.2 (Pin_2)
- net ADC_Thresh: no longer J106.2 (Pin_2)
- net D+: now also D102.2 (A2)
- net D-: now also D109.2 (A2)
- net GND: now also D102.1 (A1), D109.1 (A1), D110.1 (A1), D111.1 (A1), D113.1 (A1), D114.1 (A1), D115.1 (A1), D116.1 (A1)
- net NRST: now also C123.1, R106.1; no longer J108.10
- net SWDCLK: now also R104.1; no longer J108.04
- net SWDIO: now also R103.1; no longer J108.02
- net SWO: now also R105.1; no longer J108.06
- net String_1_out: now also D105.2 (A), D115.2 (A2)
- net String_2_out: now also D106.2 (A), D114.2 (A2)
- net String_3_out: now also D107.2 (A), D113.2 (A2)
- net String_4_out: now also D108.2 (A), D111.2 (A2)
- net VBUS_TVS: now also D110.2 (A2)
- net UART_TX renamed USART_TX
- new net: C123.2, D101.1 (A1), D103.1 (A1), D104.1 (A1), D112.1 (A1)
- new net ADC_Mode: J105.2 (Pin_2)
- new net ADC_Slider: J106.2 (Pin_2)
- new net CONN_NRST: D101.2 (A2), J108.10, R106.2
- new net CONN_SWCLK: D104.2 (A2), J108.04, R104.2
- new net CONN_SWDIO: D112.2 (A2), J108.02, R103.2
- new net CONN_SWO: D103.2 (A2), J108.06, R105.2
- new net Conn_String_1: D105.1 (K), J102.1 (Pin_1)
- new net Conn_String_2: D106.1 (K), J102.2 (Pin_2)
- new net Conn_String_3: D107.1 (K), J102.3 (Pin_3)
- new net Conn_String_4: D108.1 (K), J102.4 (Pin_4)
Other:
- added sheet IO (io.kicad_sch)
- note added: "3.3V Working 5.3V Clamp"
- note added: "5V Working 5.5V Clamp"
- note added: "Shottkys: 230mV@100mA Reverse DC: 30V"
- note removed: "2x40 Neck PCB Input Pins"
- note removed: "710-830059082"
- note removed: "75869-107LF"
- moved on the sheet: C101, C102, C103, C104, C105, C106, C107, C108, C109, C110, C111, C112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

Commit message: rev 0.3
Parts:
- removed C123: 100n, Capacitor_SMD:C_0402_1005Metric, symbol Device:C
- removed D105, D106, D107, D108: D_Small, symbol Device:D_Small
- removed SW101: SW_SPDT, JS102011SAQN:SW_JS102011SAQN, symbol Switch:SW_SPDT
- added D101: BLUE, LED_SMD:LED_0603_1608Metric, symbol Device:LED
- added D113, D114, D115, D116: D_Small, Diode_SMD:D_SOD-323, symbol Device:D_Small
- added H101, H102, H103, H104: MountingHole, MountingHole:MountingHole_3.2mm_M3, symbol Mechanical:MountingHole
- added R101: 1k, Resistor_SMD:R_0402_1005Metric, symbol Device:R
- D102: renamed from D101; footprint (none) -> 0_Footprint_lib:PMEG3005AESFYL
- D103: renamed from D102; footprint (none) -> 0_Footprint_lib:PMEG3005AESFYL
- D104: renamed from D103; footprint (none) -> 0_Footprint_lib:PMEG3005AESFYL
- D105: renamed from D111; footprint (none) -> 0_Footprint_lib:PMEG3005AESFYL
- D106: renamed from D113; footprint (none) -> 0_Footprint_lib:PMEG3005AESFYL
- D107: renamed from D104; footprint (none) -> 0_Footprint_lib:PMEG3005AESFYL
- D108: renamed from D109; footprint (none) -> 0_Footprint_lib:PMEG3005AESFYL
- D109: renamed from D110; footprint (none) -> 0_Footprint_lib:PMEG3005AESFYL
- D110: renamed from D114; footprint (none) -> 0_Footprint_lib:PMEG3005AESFYL
- D111: renamed from D112; footprint (none) -> 0_Footprint_lib:PMEG3005AESFYL
- D112: renamed from D115; footprint (none) -> 0_Footprint_lib:PMEG3005AESFYL
- D117: renamed from D116; footprint (none) -> 0_Footprint_lib:PMEG3005AESFYL
- J101: footprint 75869_332LF:AMPHENOL_75869-332LF -> 0_Footprint_lib:AMPHENOL_75869-332LF
- J102: footprint 22292041:CONN_AE-6410-04A_MOL -> 0_Footprint_lib:CONN_AE-6410-04A_MOL
- J103, J104, J105, J106, J109: footprint 22292031:CONN_AE-6410-03A_MOL -> 0_Footprint_lib:CONN_AE-6410-03A_MOL
- J108: footprint FTSH_105_01_F_D_K:SAMTEC_FTSH-105-01-F-D-K -> 0_Footprint_lib:SAMTEC_FTSH-105-01-F-D-K
- R104: renamed from R103; footprint (none) -> Resistor_SMD:R_0402_1005Metric
- R105: renamed from R104; footprint (none) -> Resistor_SMD:R_0402_1005Metric
- R106: renamed from R105; footprint (none) -> Resistor_SMD:R_0402_1005Metric
- R107: renamed from R106; footprint (none) -> Resistor_SMD:R_0402_1005Metric
- Y101: footprint 830059082:830059082 -> Crystal:Crystal_SMD_3225-4Pin_3.2x2.5mm
- renumbered R101 to R102, R102 to R103, R107 to R108, R108 to R109
Connections:
- net ADC_Mod is gone; now on net ADC_Mode: U101.41 (PA5)
- net ADC_Thresh is gone; now on net ADC_Slider: U101.46 (PB0)
- net SW_BOOT0 is gone; now on net GND: R102.1
- net Conn_String_1: now also D112.2 (A2), D113.1 (K)
- net Conn_String_2: now also D110.2 (A2), D114.1 (K)
- net Conn_String_3: now also D106.2 (A2), D115.1 (K)
- net Conn_String_4: now also D105.2 (A2), D116.1 (K)
- net GND: now also D102.1 (A1), D104.1 (A1), D107.1 (A1), D111.1 (A1), D101.1 (K)
- net String_1_out: now also D113.2 (A); no longer D112.2 (A2)
- net String_2_out: now also D114.2 (A); no longer D110.2 (A2)
- net String_3_out: now also D115.2 (A); no longer D106.2 (A2)
- net String_4_out: now also D116.2 (A); no longer D105.2 (A2)
- net LED_OUT: now reaches U101.132 (PG15)
- net LED_OUT: now also R101.2
- net ADC_Extra: no longer names the net of U101.47 (PB1)
- net USART_TX renamed UART_TX
- new net LED_BLUE: D101.2 (A), R101.1
Other:
- moved on the sheet: C106, D105, D106, D110, D112

Commit message: rev 0.4
Connections:
- net LED_OUT: now also U101.74 (PB13); no longer U101.132 (PG15)
- net input_1: now also U101.13 (PF3); no longer U101.100 (PA8)
- net input_10: now also U101.1 (PE2); no longer U101.27 (PC1)
- net input_11: now also U101.54 (PF14); no longer U101.28 (PC2)
- net input_12: now also U101.53 (PF13); no longer U101.29 (PC3)
- net input_13: now also U101.50 (PF12); no longer U101.44 (PC4)
- net input_14: now also U101.49 (PF11); no longer U101.45 (PC5)
- net input_15: now also U101.45 (PC5); no longer U101.96 (PC6)
- net input_16: now also U101.44 (PC4); no longer U101.97 (PC7)
- net input_17: now also U101.29 (PC3); no longer U101.98 (PC8)
- net input_18: now also U101.28 (PC2); no longer U101.99 (PC9)
- net input_19: now also U101.27 (PC1); no longer U101.111 (PC10)
- net input_2: now also U101.14 (PF4); no longer U101.102 (PA10)
- net input_20: now also U101.22 (PF10); no longer U101.112 (PC11)
- net input_21: now also U101.19 (PF7); no longer U101.113 (PC12)
- net input_22: now also U101.21 (PF9); no longer U101.7 (PC13)
- net input_23: now also U101.20 (PF8); no longer U101.8 (PC14)
- net input_24: now also U101.18 (PF6); no longer U101.9 (PC15)
- net input_25: now also U101.15 (PF5); no longer U101.114 (PD0)
- net input_26: now also U101.11 (PF1); no longer U101.115 (PD1)
- net input_27: now also U101.8 (PC14); no longer U101.116 (PD2)
- net input_28: now also U101.7 (PC13); no longer U101.117 (PD3)
- net input_29: now also U101.5 (PE6); no longer U101.118 (PD4)
- net input_3: now also U101.10 (PF0); no longer U101.110 (PA15)
- net input_30: now also U101.142 (PE1); no longer U101.119 (PD5)
- net input_31: now also U101.141 (PE0); no longer U101.122 (PD6)
- net input_32: now also U101.139 (PB8); no longer U101.123 (PD7)
- net input_33: now also U101.140 (PB9); no longer U101.78 (PD9)
- net input_34: now also U101.137 (PB7); no longer U101.79 (PD10)
- net input_35: now also U101.136 (PB6); no longer U101.80 (PD11)
- net input_36: now also U101.135 (PB5); no longer U101.81 (PD12)
- net input_37: now also U101.134 (PB4); no longer U101.82 (PD13)
- net input_38: now also U101.129 (PG14); no longer U101.85 (PD14)
- net input_39: now also U101.124 (PG9); no longer U101.86 (PD15)
- net input_4: now also U101.12 (PF2); no longer U101.69 (PB10)
- net input_40: now also U101.123 (PD7); no longer U101.1 (PE2)
- net input_41: now also U101.57 (PG1); no longer U101.2 (PE3)
- net input_42: now also U101.55 (PF15); no longer U101.3 (PE4)
- net input_43: now also U101.59 (PE8); no longer U101.4 (PE5)
- net input_44: now also U101.58 (PE7); no longer U101.5 (PE6)
- net input_45: now also U101.63 (PE10); no longer U101.58 (PE7)
- net input_46: now also U101.60 (PE9); no longer U101.59 (PE8)
- net input_47: now also U101.66 (PE13); no longer U101.60 (PE9)
- net input_48: now also U101.64 (PE11); no longer U101.63 (PE10)
- net input_49: now also U101.65 (PE12); no longer U101.64 (PE11)
- net input_5: now also U101.4 (PE5); no longer U101.70 (PB11)
- net input_50: now also U101.68 (PE15); no longer U101.65 (PE12)
- net input_51: now also U101.69 (PB10); no longer U101.66 (PE13)
- net input_53: now also U101.73 (PB12); no longer U101.68 (PE15)
- net input_54: now also U101.70 (PB11); no longer U101.10 (PF0)
- net input_55: now also U101.76 (PB15); no longer U101.11 (PF1)
- net input_56: now also U101.75 (PB14); no longer U101.12 (PF2)
- net input_57: now also U101.82 (PD13); no longer U101.13 (PF3)
- net input_58: now also U101.78 (PD9); no longer U101.14 (PF4)
- net input_59: now also U101.86 (PD15); no longer U101.15 (PF5)
- net input_6: now also U101.9 (PC15); no longer U101.73 (PB12)
- net input_60: now also U101.85 (PD14); no longer U101.18 (PF6)
- net input_61: now also U101.90 (PG5); no longer U101.19 (PF7)
- net input_62: now also U101.88 (PG3); no longer U101.20 (PF8)
- net input_63: now also U101.93 (PG8); no longer U101.21 (PF9)
- net input_64: now also U101.92 (PG7); no longer U101.22 (PF10)
- net input_65: now also U101.98 (PC8); no longer U101.49 (PF11)
- net input_66: now also U101.96 (PC6); no longer U101.50 (PF12)
- net input_67: now also U101.100 (PA8); no longer U101.53 (PF13)
- net input_68: now also U101.99 (PC9); no longer U101.54 (PF14)
- net input_69: now also U101.110 (PA15); no longer U101.55 (PF15)
- net input_7: now also U101.2 (PE3); no longer U101.74 (PB13)
- net input_70: now also U101.102 (PA10); no longer U101.56 (PG0)
- net input_71: now also U101.112 (PC11); no longer U101.57 (PG1)
- net input_72: now also U101.111 (PC10); no longer U101.87 (PG2)
- net input_73: now also U101.114 (PD0); no longer U101.88 (PG3)
- net input_74: now also U101.113 (PC12); no longer U101.89 (PG4)
- net input_75: now also U101.116 (PD2); no longer U101.90 (PG5)
- net input_76: now also U101.115 (PD1); no longer U101.91 (PG6)
- net input_77: now also U101.118 (PD4); no longer U101.92 (PG7)
- net input_78: now also U101.117 (PD3); no longer U101.93 (PG8)
- net input_79: now also U101.122 (PD6); no longer U101.124 (PG9)
- net input_8: now also U101.3 (PE4); no longer U101.75 (PB14)
- net input_80: now also U101.119 (PD5); no longer U101.129 (PG14)
- net input_9: now also U101.56 (PG0); no longer U101.76 (PB15)

Commit message: rev1.02
Parts:
- D109: value D_TVS_Small -> D_TVS_VBUS
- U101: now left out of the parts list
Changed lines of the file:
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@@
 			)
 		)
-		(property "Value" "D_TVS_Small"
+		(property "Value" "D_TVS_VBUS"
 			(at 308.61 46.9899 90)
 			(effects
@@
 		(unit 1)
 		(exclude_from_sim no)
-		(in_bom yes)
+		(in_bom no)
 		(on_board yes)
 		(dnp no)

Commit message: rev 1.04
- gerbers/BOM/CPL files are all generated.
Parts:
- C101: JLCPCB Part # (none) -> C19702
- C102, C103, C104, C105, C106, C107, C109, C110, C111, C113, C115, C116, C118, C119: JLCPCB Part # (none) -> C1525
- C108, C112: value 10p -> 12p; JLCPCB Part # (none) -> C161304
- C114, C117: footprint Capacitor_SMD:C_0402_1005Metric -> Capacitor_SMD:C_0603_1608Metric; JLCPCB Part # (none) -> C99228
- C120: JLCPCB Part # (none) -> C60133
- C121, C122: JLCPCB Part # (none) -> C52923
- D101: JLCPCB Part # (none) -> C2288
- D102, D103, D104, D105, D106, D107, D108, D110, D111, D112, D117: JLCPCB Part # (none) -> C2908830
- D109: JLCPCB Part # (none) -> C2443412
- D113, D114, D115, D116: JLCPCB Part # (none) -> C146335
- FB101: JLCPCB Part # (none) -> C113030
- H101, H102, H103, H104, U101: now not fitted
- J101, J102, J103, J104, J105, J106, J107, J108, J109: now not fitted; now left out of the parts list
- R101: JLCPCB Part # (none) -> C11702
- R102, R103: JLCPCB Part # (none) -> C17902
- R104, R105, R106, R107: JLCPCB Part # (none) -> C25092
- R108: JLCPCB Part # (none) -> C25779
- R109: JLCPCB Part # (none) -> C4142
- Y101: JLCPCB Part # (none) -> C13738
Other:
- note added: "90 Ohm @ 0.286mm Width, 2.032mm Space"
