File: ControllerPCB/Power.kicad_sch (KiCad schematic)
At the start: 11 parts, among them J201 9V Humbucker OUT, J202 9V IN, U201 ADP3336ARMZ

Commit message: rev 0.3
Parts:
- D201: footprint (none) -> 0_Footprint_lib:PMEG3005AESFYL
- J201: footprint 3_641126_2:TE_3-641126-2 -> 0_Footprint_lib:TE_3-641126-2
- J202: footprint PowerConnector:APP_ASMPR45-1X2-RK -> 0_Footprint_lib:APP_ASMPR45-1X2-RK
- U201: footprint ADP3336ARMZ_REEL7:RM_8_ADI -> 0_Footprint_lib:RM_8_ADI
Connections:
- net 9V+ is gone; now on net GND: C201.1, D201.2 (A2), J202.1, U201.6 (~{SD}), U201.7 (IN), U201.8 (IN)
- net GND: now also J201.1 (Pin_1), J201.2 (Pin_2)
- net FB_IN: now reaches C202.2, R201.2, R202.1, U201.5 (FB)
- net LED_GREEN: now reaches D202.1 (K), R203.1
Other:
- note removed: "some sort of decoupling here"
- moved on the sheet: J201
Changed lines of the file:
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@@
+	)
+	(junction
+		(at 49.53 55.88)
+		(diameter 0)
+		(color 0 0 0 0)
 	)
 	(junction
@@
 	)
 	(junction
+		(at 50.8 58.42)
+		(diameter 0)
+		(color 0 0 0 0)
+	)
+	(junction
 		(at 116.84 58.42)
 		(diameter 0)
@@
 	(wire
 		(pts
+			(xy 50.8 58.42) (xy 58.42 58.42)
+		)
+		(stroke
+			(width 0)
+			(type default)
+		)
+	)
+	(wire
+		(pts
 			(xy 74.93 49.53) (xy 74.93 53.34)
 		)
@@
 	(wire
 		(pts
-			(xy 48.26 55.88) (xy 58.42 55.88)
+			(xy 48.26 55.88) (xy 49.53 55.88)
 		)
 		(stroke
@@
 	(wire
 		(pts
+			(xy 49.53 55.88) (xy 58.42 55.88)
+		)
+		(stroke
+			(width 0)
+			(type default)
+		)
+	)
+	(wire
+		(pts
 			(xy 58.42 55.88) (xy 58.42 49.53)
 		)
@@
 	(wire
 		(pts
+			(xy 49.53 68.58) (xy 49.53 55.88)
+		)
+		(stroke
+			(width 0)
+			(type default)
+		)
+	)
+	(wire
+		(pts
 			(xy 64.77 68.58) (xy 74.93 68.58)
 		)
@@
 	(wire
 		(pts
+			(xy 41.91 68.58) (xy 49.53 68.58)
+		)
+		(stroke
+			(width 0)
+			(type default)
+		)
+	)
+	(wire
+		(pts
 			(xy 64.77 49.53) (xy 64.77 54.61)
 		)
@@
 	(wire
 		(pts
-			(xy 48.26 58.42) (xy 58.42 58.42)
+			(xy 48.26 58.42) (xy 50.8 58.42)
 		)
 		(stroke
@@
 	(wire
 		(pts
+			(xy 41.91 71.12) (xy 50.8 71.12)
+		)
+		(stroke
+			(width 0)
+			(type default)
+		)
+	)
+	(wire
+		(pts
+			(xy 50.8 71.12) (xy 50.8 58.42)
+		)
+		(stroke
+			(width 0)
+			(type default)
+		)
+	)
+	(wire
+		(pts
 			(xy 58.42 68.58) (xy 64.77 68.58)
 		)
@@
 		)
 	)
-	(text "some sort of decoupling here\n"
-		(exclude_from_sim no)
-		(at 37.592 80.264 0)
+	(label "FB_IN"
+		(at 110.49 58.42 0)
+		(effects
+			(font
+				(size 0.889 0.889)
+			)
+			(justify left bottom)
+		)
+	)
+	(label "V_DIV"
+		(at 120.65 58.42 0)
+		(effects
+			(font
+				(size 0.889 0.889)
+			)
+			(justify left bottom)
+		)
+	)
+	(label "9V-"
+		(at 49.53 58.42 0)
 		(effects
 			(font
 				(size 1.27 1.27)
 			)
-		)
-	)
-	(label "9V-"
-		(at 49.53 58.42 0)
+			(justify left bottom)
+		)
+	)
+	(label "LED_GREEN"
+		(at 160.02 49.53 0)
 		(effects
 			(font
@@
 			)
 		)
-		(property "Footprint" ""
+		(property "Footprint" "0_Footprint_lib:PMEG3005AESFYL"
 			(at 64.77 57.15 0)
 			(effects
@@
 			)
 		)
-		(property "Footprint" "ADP3336ARMZ_REEL7:RM_8_ADI"
+		(property "Footprint" "0_Footprint_lib:RM_8_ADI"
 			(at 119.38 62.23 0)
 			(effects
@@
 	(symbol
 		(lib_id "Connector:Conn_01x02_Pin")
-		(at 35.56 73.66 0)
+		(at 36.83 68.58 0)
 		(unit 1)
 		(exclude_from_sim no)
@@
 		(dnp no)
 		(property "Reference" "J201"
-			(at 36.068 67.818 0)
+			(at 37.338 62.738 0)
 			(effects
 				(font
@@
 		)
 		(property "Value" "9V Humbucker OUT"
-			(at 36.322 70.612 0)
+			(at 37.592 65.532 0)
 			(effects
 				(font
@@
 			)
 		)
-		(property "Footprint" "3_641126_2:TE_3-641126-2"
-			(at 35.56 73.66 0)
+		(property "Footprint" "0_Footprint_lib:TE_3-641126-2"
+			(at 36.83 68.58 0)
 			(effects
 				(font
@@
 		)
 		(property "Datasheet" "~"
-			(at 35.56 73.66 0)
+			(at 36.83 68.58 0)
 			(effects
 				(font
@@
 		)
 		(property "Description" "Generic connector, single row, 01x02, script generated"
-			(at 35.56 73.66 0)
+			(at 36.83 68.58 0)
 			(effects
 				(font
@@
 			)
 		)
-		(property "Footprint" "PowerConnector:APP_ASMPR45-1X2-RK"
+		(property "Footprint" "0_Footprint_lib:APP_ASMPR45-1X2-RK"
 			(at 38.1 55.88 0)
 			(effects

Commit message: rev 1.04
- gerbers/BOM/CPL files are all generated.
Parts:
- C201, C203: JLCPCB Part # (none) -> C52923
- C202: JLCPCB Part # (none) -> C1546
- D201: JLCPCB Part # (none) -> C2908830
- D202: JLCPCB Part # (none) -> C22371297
- J201, J202, U201: now not fitted; now left out of the parts list
- R201: JLCPCB Part # (none) -> C2998127
- R202: JLCPCB Part # (none) -> C852915
- R203: JLCPCB Part # (none) -> C11702
Changed lines of the file:
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@@
+			)
+		)
+		(property "JLCPCB Part #" "C52923"
+			(at 74.93 57.15 0)
+			(effects
+				(font
+					(size 1.27 1.27)
+				)
+				(hide yes)
 			)
 		)
@@
 			)
 		)
+		(property "JLCPCB Part #" "C2998127"
+			(at 127 53.34 0)
+			(effects
+				(font
+					(size 1.27 1.27)
+				)
+				(hide yes)
+			)
+		)
 		(pin "2"
 		)
@@
 			)
 		)
+		(property "JLCPCB Part #" "C2908830"
+			(at 64.77 57.15 0)
+			(effects
+				(font
+					(size 1.27 1.27)
+				)
+				(hide yes)
+			)
+		)
 		(pin "2"
 		)
@@
 		)
 		(property "Description" "Unpolarized capacitor"
+			(at 116.84 53.34 0)
+			(effects
+				(font
+					(size 1.27 1.27)
+				)
+				(hide yes)
+			)
+		)
+		(property "JLCPCB Part #" "C1546"
 			(at 116.84 53.34 0)
 			(effects
@@
 			)
 		)
+		(property "JLCPCB Part #" "C11702 "
+			(at 163.83 59.69 0)
+			(effects
+				(font
+					(size 1.27 1.27)
+				)
+				(hide yes)
+			)
+		)
 		(pin "2"
 		)
@@
 		(unit 1)
 		(exclude_from_sim no)
-		(in_bom yes)
-		(on_board yes)
-		(dnp no)
+		(in_bom no)
+		(on_board yes)
+		(dnp yes)
 		(fields_autoplaced yes)
 		(property "Reference" "U201"
@@
 		)
 		(property "Description" "High Accuracy Ultralow IQ, 500mA anyCAP Adjustable Low Dropout Regulator, MSOP-8"
+			(at 99.06 52.07 0)
+			(effects
+				(font
+					(size 1.27 1.27)
+				)
+				(hide yes)
+			)
+		)
+		(property "JLCPCB Part #" ""
 			(at 99.06 52.07 0)
 			(effects
@@
 			)
 		)
+		(property "JLCPCB Part #" "C52923"
+			(at 143.51 57.15 0)
+			(effects
+				(font
+					(size 1.27 1.27)
+				)
+				(hide yes)
+			)
+		)
 		(pin "1"
 		)
@@
 			)
 		)
+		(property "JLCPCB Part #" "C22371297"
+			(at 154.94 49.53 0)
+			(effects
+				(font
+					(size 1.27 1.27)
+				)
+				(hide yes)
+			)
+		)
 		(pin "2"
 		)
@@
 		(unit 1)
 		(exclude_from_sim no)
-		(in_bom yes)
-		(on_board yes)
-		(dnp no)
+		(in_bom no)
+		(on_board yes)
+		(dnp yes)
 		(property "Reference" "J201"
 			(at 37.338 62.738 0)
@@
 		)
 		(property "Description" "Generic connector, single row, 01x02, script generated"
+			(at 36.83 68.58 0)
+			(effects
+				(font
+					(size 1.27 1.27)
+				)
+				(hide yes)
+			)
+		)
+		(property "JLCPCB Part #" ""
 			(at 36.83 68.58 0)
 			(effects
@@
 			)
 		)
+		(property "JLCPCB Part #" "C852915"
+			(at 127 63.5 0)
+			(effects
+				(font
+					(size 1.27 1.27)
+				)
+				(hide yes)
+			)
+		)
 		(pin "1"
 		)
@@
 		(unit 1)
 		(exclude_from_sim no)
-		(in_bom yes)
-		(on_board yes)
-		(dnp no)
+		(in_bom no)
+		(on_board yes)
+		(dnp yes)
 		(property "Reference" "J202"
 			(at 37.846 49.53 0)
@@
 				(hide yes)
 			)
+		)
+		(property "JLCPCB Part #" ""
+			(at 38.1 55.88 0)
+			(effects
+				(font
+					(size 1.27 1.27)
+				)
+				(hide yes)
+			)
