File: ControllerPCB/io.kicad_sch (KiCad schematic)
At the start: 82 parts, among them J501 2x20 Conn_1, J502 2x20 Conn_2

Commit message: rev 1.04
- gerbers/BOM/CPL files are all generated.
Parts:
- D501, D502, D503, D504, D505, D506, D507, D508, D509, D510, D511, D512, D513, D514, D515, D516, D517, D518, D519, D520, D521, D522, D523, D524, D525, D526, D527, D528, D529, D530, D531, D532, D533, D534, D535, D536, D537, D538, D539, D540, D541, D542, D543, D544, D545, D546, D547, D548, D549, D550, D551, D552, D553, D554, D555, D556, D557, D558, D559, D560, D561, D562, D563, D564, D565, D566, D567, D568, D569, D570, D571, D572, D573, D574, D575, D576, D577, D578, D579, D580: JLCPCB Part # (none) -> C2908830
- J501, J502: now not fitted; now left out of the parts list
